File: update.kicad_pcb (KiCad board)
At the start: 2 copper layers, 2.5 x 6 mm, 23 parts, among them J1 PJ-037A, M1 Fan (MF40101V1-1000U-A99), Q1 2N3055, U1 LM7812_TO220, U2 TPS54302, U3 LM723CN

Commit message: update
Parts:
- C1, C3: footprint Library:CAP_CL10_SAM -> Capacitor_SMD:C_0603_1608Metric
- C2: footprint Library:CAP_CL32A_SAM -> Capacitor_SMD:C_0603_1608Metric
- C4, C5: footprint Library:CAP_GRM_P6XP3_MUR -> Capacitor_SMD:C_0603_1608Metric
- C6, C7: footprint Library:CAP_3216_TDK -> Capacitor_SMD:C_0603_1608Metric
- C9: footprint Library:CAP_04025C101JAT2A -> Capacitor_SMD:C_0603_1608Metric
- L1: footprint Library:IND_AMRU00060630100MA1_CHE -> Inductor_SMD:L_0603_1608Metric
- LED1: footprint Library:LED_5988A10107F_DIA -> LED_SMD:LED_0603_1608Metric
- R2, R3, R5: footprint Library:RC0603N_YAG -> Resistor_SMD:R_0603_1608Metric
- R4: footprint Library:RES_RC0603_YAG -> Resistor_SMD:R_0603_1608Metric
- moved J1 72.2 mm to (201.0, 108.0)
- moved C2 66.4 mm to (202.2, 65.0)
- moved C6 62.1 mm to (184.8, 76.0)
- moved C3 52.1 mm to (177.2, 65.0)
- moved C4 45.7 mm to (202.2, 68.0)
- moved R2 39.7 mm to (202.2, 72.0)
- moved U2 39.4 mm to (185.1, 66.0)
- moved R3 39.3 mm to (202.2, 75.0)
- moved R4 28.4 mm to (202.2, 78.0)
- moved C5 23.8 mm to (185.2, 73.0)
- moved C8 20.8 mm to (185.2, 80.0)
- moved U3 14.0 mm to (124.4, 102.5)

Commit message: layout update
Parts:
- C2: value CL32A106KLULNNE -> 10uF
- C4, C5: value GRM033R6YA104KE14D -> 0.1uF
- C6, C7: value C3216X5R1V226M160AC -> 22uF
- C8: value GRM0335C1H750JA01D -> 75pF
- L1: value AMRU00060630100MA1 -> 10uH
- M1: moved to B.Cu
- R2: value RC0603FR-07511KL -> 511kΩ
- R3: value RC0603FR-07105KL -> 105kΩ
- R4: value RC0603FR-1349R9L -> 49.9Ω
- moved C9 60.2 mm to (179.4, 101.1)
- moved C1 58.7 mm to (192.2, 79.8), turned to -90 degrees
- moved U1 58.3 mm to (195.1, 78.6), turned to -90 degrees
- moved C2 52.2 mm to (152.6, 81.2), turned to -90 degrees
- moved C4 48.7 mm to (155.3, 81.2), turned to -90 degrees
- moved C7 44.7 mm to (160.4, 86.2)
- moved L1 43.0 mm to (148.5, 79.7), turned to -90 degrees
- moved U3 41.7 mm to (165.6, 96.0)
- moved C8 36.0 mm to (149.3, 77.0), turned to 180 degrees
- moved R3 34.3 mm to (168.4, 81.3), turned to 90 degrees
- moved R2 32.8 mm to (170.8, 81.3), turned to -90 degrees
- moved R4 32.5 mm to (169.7, 78.7)
- moved LED1 31.9 mm to (188.5, 78.4), turned to 90 degrees
- moved R5 31.6 mm to (179.2, 105.1)
- moved M1 29.2 mm to (186.2, 84.3)
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Routing:
- net Net-(U2-BOOT): track 0.00 -> 6.63 mm
- net +24V: track 6.01 -> 0.14 mm
- net GND: track 6.41 -> 1.97 mm
- net /NInverting: track 0.00 -> 2.97 mm
- net (no net): vias 0 -> 12
- added copper zone on F.Cu, net (none)
- added copper zone on F.Cu, net +12V
- added copper zone on F.Cu, net +24V
- added copper zone on F.Cu, net GND
