File: v3/v3.kicad_sch (KiCad schematic)
At the start: 25 parts, among them J1 PJ-037A, M1 Fan (MF40101V1-1000U-A99), Q1 2N3055, U1 LM7812_TO220, U2 TPS54302, U3 LM723CN

Commit message: v3_latest
Parts:
- removed C9: 04025C501KAT2A, Capacitor_SMD:C_0603_1608Metric, symbol 2024-01-13_05-40-23:04025C501KAT2A
- removed J1: PJ-037A, CONN1x2_PJ-037A_CUD, symbol 2024-01-14_16-39-54:PJ-037A
- added C10: 500pF50VX7R, Capacitor_SMD:C_0603_1608Metric, symbol 2024-01-20_01-26-05:CC0603KRX7R9BB501
- added J2: PJ-037A, Library:CUI_PJ-037A, symbol PJ-037A:PJ-037A
- C1, C3: value CL10A105KL8NNNC -> 1uF35VX5R
- C4, C5: value GRM033R6YA104KE14D -> 0.1uF35VX5R
- C8: value GRM0335C1H750JA01D -> 75pF50VC0G
- L1: value AMRU00060630100MA1 -> 10uH
- R1: value RN73R2ATTD2081A10 -> 2.08K
- R2: value RC0603FR-07511KL -> 511K
- R3: value RC0603FR-07105KL -> 105K
- R4: value RC0603FR-1349R9L -> 49.9R
- R5: value RC0603FR-0710RL -> 10R
Connections:
- net +24V: now also J2.1
- net GND: now also J2.2
- net comp: now also C10.1
- net at R7.2: now also C10.2
Changed lines of the file:
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@@
+    (stroke (width 0) (type default))
+  )
+  (wire (pts (xy 57.15 55.88) (xy 57.15 57.15))
     (stroke (width 0) (type default))
   )
@@
     (stroke (width 0) (type default))
   )
+  (wire (pts (xy 57.15 53.34) (xy 57.15 52.07))
+    (stroke (width 0) (type default))
+  )
   (wire (pts (xy 130.81 130.81) (xy 144.78 130.81))
     (stroke (width 0) (type default))
@@
     (stroke (width 0) (type default))
   )
-  (wire (pts (xy 71.12 55.88) (xy 58.42 55.88))
+  (wire (pts (xy 57.15 55.88) (xy 71.12 55.88))
     (stroke (width 0) (type default))
   )
@@
     (stroke (width 0) (type default))
   )
-  (wire (pts (xy 58.42 53.34) (xy 69.85 53.34))
+  (wire (pts (xy 57.15 53.34) (xy 69.85 53.34))
     (stroke (width 0) (type default))
   )
@@
       (effects (font (size 1.27 1.27)) (justify right))
     )
-    (property "Value" "RN73R2ATTD2081A10" (at 107.95 111.76 0)
+    (property "Value" "2.08K" (at 107.95 111.76 0)
       (effects (font (size 0.7 0.7)) (justify right))
     )
@@
       (effects (font (size 0.7 0.7)))
     )
-    (property "Value" "CL10A105KL8NNNC" (at 52.07 118.11 0)
+    (property "Value" "1uF35VX5R" (at 52.07 118.11 0)
       (effects (font (size 0.7 0.7)))
     )
@@
       (effects (font (size 1.524 1.524)) (justify right))
     )
-    (property "Value" "RC0603FR-07511KL" (at 111.76 40.64 90)
+    (property "Value" "511K" (at 111.76 40.64 90)
       (effects (font (size 0.7 0.7)) (justify right))
     )
@@
       (effects (font (size 1.524 1.524)) (justify right))
     )
-    (property "Value" "RC0603FR-07105KL" (at 113.03 60.96 90)
+    (property "Value" "105K" (at 113.03 60.96 90)
       (effects (font (size 1.524 1.524)) (justify right))
     )
@@
       (effects (font (size 1.524 1.524)) (justify right))
     )
-    (property "Value" "GRM033R6YA104KE14D" (at 96.52 41.91 90)
+    (property "Value" "0.1uF35VX5R" (at 96.52 41.91 90)
       (effects (font (size 0.7 0.7)) (justify right))
     )
@@
       (effects (font (size 1.524 1.524)))
     )
-    (property "Value" "AMRU00060630100MA1" (at 168.91 36.83 0)
+    (property "Value" "10uH" (at 168.91 36.83 0)
       (effects (font (size 0.7 0.7)))
     )
@@
       (effects (font (size 1.524 1.524)) (justify right))
     )
-    (property "Value" "RC0603FR-1349R9L" (at 213.36 52.07 90)
+    (property "Value" "49.9R" (at 213.36 52.07 90)
       (effects (font (size 0.7 0.7)) (justify right))
     )
@@
     )
   )
+  (symbol (lib_id "2024-01-20_01-26-05:CC0603KRX7R9BB501") (at 208.28 163.83 0) (unit 1)
+    (in_bom yes) (on_board yes) (dnp no) (fields_autoplaced)
+    (property "Reference" "C10" (at 212.09 157.48 0)
+      (effects (font (size 1.524 1.524)))
+    )
+    (property "Value" "500pF50VX7R" (at 212.09 160.02 0)
+      (effects (font (size 1.524 1.524)))
+    )
+    (property "Footprint" "Capacitor_SMD:C_0603_1608Metric" (at 208.28 163.83 0)
+      (effects (font (size 1.27 1.27) italic) hide)
+    )
+    (property "Datasheet" "CC0603KRX7R9BB501" (at 208.28 163.83 0)
+      (effects (font (size 1.27 1.27) italic) hide)
+    )
+    (pin "1")
+    (pin "2")
+    (instances
+      (project "v3"
+        (path "/43152005-bbce-4fe9-aacf-31369492adcb"
+          (reference "C10") (unit 1)
+        )
+      )
+    )
+  )
   (symbol (lib_id "2024-01-14_22-06-53:RC0603FR-0710RL") (at 226.06 134.62 90) (unit 1)
     (in_bom yes) (on_board yes) (dnp no) (fields_autoplaced)
@@
       (effects (font (size 1.524 1.524)) (justify right))
     )
-    (property "Value" "RC0603FR-0710RL" (at 228.6 129.54 90)
+    (property "Value" "10R" (at 228.6 129.54 90)
       (effects (font (size 0.7 0.7)) (justify right))
     )
@@
       (effects (font (size 1.27 1.27)) (justify right))
     )
-    (property "Value" "GRM0335C1H750JA01D" (at 200.66 85.09 0)
+    (property "Value" "75pF50VC0G" (at 200.66 85.09 0)
       (effects (font (size 0.7 0.7)) (justify right))
     )
@@
         (path "/827be695-0790-4bef-8095-9451fa66e5ff"
           (reference "C8") (unit 1)
-        )
-      )
-    )
-  )
-  (symbol (lib_id "2024-01-13_05-40-23:04025C501KAT2A") (at 208.28 163.83 0) (unit 1)
-    (in_bom yes) (on_board yes) (dnp no)
-    (property "Reference" "C9" (at 212.09 160.02 0)
-      (effects (font (size 1.524 1.524)))
-    )
-    (property "Value" "04025C501KAT2A" (at 212.09 166.37 0)
-      (effects (font (size 0.7 0.7)))
-    )
-    (property "Footprint" "Capacitor_SMD:C_0603_1608Metric" (at 208.28 163.83 0)
-      (effects (font (size 1.27 1.27) italic) hide)
-    )
-    (property "Datasheet" "04025C501KAT2A" (at 208.28 163.83 0)
-      (effects (font (size 1.27 1.27) italic) hide)
-    )
-    (pin "1")
-    (pin "2")
-    (instances
-      (project "v3"
-        (path "/43152005-bbce-4fe9-aacf-31369492adcb"
-          (reference "C9") (unit 1)
-        )
-      )
-      (project "Schematic2"
-        (path "/80952055-fa96-4634-8dc0-154c3a08535a"
-          (reference "C1") (unit 1)
-        )
-      )
-      (project "update"
-        (path "/827be695-0790-4bef-8095-9451fa66e5ff"
-          (reference "C9") (unit 1)
         )
       )
@@
     )
   )
-  (symbol (lib_id "2024-01-14_16-39-54:PJ-037A") (at 58.42 55.88 180) (unit 1)
-    (in_bom yes) (on_board yes) (dnp no) (fields_autoplaced)
-    (property "Reference" "J1" (at 49.53 45.72 0)
-      (effects (font (size 1.524 1.524)))
-    )
-    (property "Value" "PJ-037A" (at 49.53 48.26 0)
-      (effects (font (size 1.524 1.524)))
-    )
-    (property "Footprint" "CONN1x2_PJ-037A_CUD" (at 58.42 55.88 0)
-      (effects (font (size 1.27 1.27) italic) hide)
-    )
-    (property "Datasheet" "PJ-037A" (at 58.42 55.88 0)
-      (effects (font (size 1.27 1.27) italic) hide)
-    )
-    (pin "1")
-    (pin "2")
-    (instances
-      (project "v3"
-        (path "/43152005-bbce-4fe9-aacf-31369492adcb"
-          (reference "J1") (unit 1)
-        )
-      )
-      (project "Schematic2"
-        (path "/80952055-fa96-4634-8dc0-154c3a08535a"
-          (reference "J2") (unit 1)
-        )
-      )
-      (project "update"
-        (path "/827be695-0790-4bef-8095-9451fa66e5ff"
-          (reference "J1") (unit 1)
-        )
-      )
-    )
-  )
   (symbol (lib_id "power:+24V") (at 71.12 52.07 270) (unit 1)
     (in_bom yes) (on_board yes) (dnp no)
@@
         (path "/827be695-0790-4bef-8095-9451fa66e5ff"
           (reference "M1") (unit 1)
+        )
+      )
+    )
+  )
+  (symbol (lib_id "PJ-037A:PJ-037A") (at 52.07 54.61 0) (unit 1)
+    (in_bom yes) (on_board yes) (dnp no) (fields_autoplaced)
+    (property "Reference" "J2" (at 48.5802 45.72 0)
+      (effects (font (size 1.27 1.27)))
+    )
+    (property "Value" "PJ-037A" (at 48.5802 48.26 0)
+      (effects (font (size 1.27 1.27)))
+    )
+    (property "Footprint" "Library:CUI_PJ-037A" (at 52.07 54.61 0)
+      (effects (font (size 1.27 1.27)) (justify bottom) hide)
+    )
+    (property "Datasheet" "" (at 52.07 54.61 0)
+      (effects (font (size 1.27 1.27)) hide)
+    )
+    (property "MANUFACTURER" "CUI INC" (at 52.07 54.61 0)
+      (effects (font (size 1.27 1.27)) (justify bottom) hide)
+    )
+    (property "STANDARD" "Manufacturer recommendations" (at 52.07 54.61 0)
+      (effects (font (size 1.27 1.27)) (justify bottom) hide)
+    )
+    (pin "1")
+    (pin "2")
+    (instances
+      (project "v3"
+        (path "/43152005-bbce-4fe9-aacf-31369492adcb"
+          (reference "J2") (unit 1)
         )
       )
@@
       (effects (font (size 0.7 0.7)))
     )
-    (property "Value" "CL10A105KL8NNNC" (at 97.79 115.57 0)
+    (property "Value" "1uF35VX5R" (at 97.79 115.57 0)
       (effects (font (size 0.7 0.7)))
     )
@@
       (effects (font (size 1.524 1.524)) (justify right))
     )
-    (property "Value" "GRM033R6YA104KE14D" (at 146.05 27.94 0)
+    (property "Value" "0.1uF35VX5R" (at 146.05 27.94 0)
       (effects (font (size 0.7 0.7)) (justify right))
     )
