File: v3/v3.kicad_pcb (KiCad board)
At the start: 2 copper layers, 72.9 x 60.9 mm, 25 parts, among them J1 PJ-037A, M1 Fan (MF40101V1-1000U-A99), Q1 2N3055, U1 LM7812_TO220, U2 TPS54302, U3 LM723CN

Commit message: v3_latest
Parts:
- removed C9: 04025C501KAT2A, Capacitor_SMD:C_0603_1608Metric
- removed J1: PJ-037A, Library:CONN1x2_PJ-037A_CUD
- added C10: 500pF50VX7R, Capacitor_SMD:C_0603_1608Metric, F.Cu at (197.1, 59.6)
- added J2: PJ-037A, Library:CUI_PJ-037A, F.Cu at (209.9, 84.0)
- C1, C3: value CL10A105KL8NNNC -> 1uF35VX5R
- C4, C5: value GRM033R6YA104KE14D -> 0.1uF35VX5R
- C8: value GRM0335C1H750JA01D -> 75pF50VC0G
- L1: value AMRU00060630100MA1 -> 10uH
- R2: value RC0603FR-07511KL -> 511K
- R3: value RC0603FR-07105KL -> 105K
- R4: value RC0603FR-1349R9L -> 49.9R
- R5: value RC0603FR-0710RL -> 10R
Routing:
- net +24V: track 44.8 -> 37.9 mm
- net GND: track 163.4 -> 161.1 mm, vias 14 -> 12

Commit message: v3_latest
Parts:
- added REF**: EdgertonLogo, Library:EdgertonLogo, F.Cu at (207.4, 51.5)
- added REF**: MechELogo, Library:MechELogo, F.Cu at (207.9, 43.3)
Other:
- board text added: "Designed by Kanishk Pal"
